Commit message: add duckieboat

File: vrx_ws/src/vrx/wamv_description/urdf/thrusters/engine.xacro (robot description, xacro)
@@ -1,3 +1,3 @@
-<?xml version="1.0"?>
+<?xml version="1.0" ?>
 <robot xmlns:xacro="http://ros.org/wiki/xacro" name="wam-v-two-engines">
   <!-- Macro for inserting an engine with its propeller. -->
@@ -6,5 +6,5 @@
       <visual>
         <geometry>
-          <mesh filename="package://wamv_description/models/engine/mesh/engine.dae"/>
+          <mesh filename="package://wamv_description/models/engine/mesh/engine.dae" />
         </geometry>
       </visual>
@@ -22,6 +22,6 @@
       </collision>
       <inertial>
-        <mass value="15"/>
-        <inertia ixx="0.889245" ixy="0.0" ixz="0.0" iyy="0.911125" iyz="0.0" izz="0.078125"/>
+        <mass value="15" />
+        <inertia ixx="0.889245" ixy="0.0" ixz="0.0" iyy="0.911125" iyz="0.0" izz="0.078125" />
       </inertial>
     </link>
@@ -29,5 +29,5 @@
       <visual>
         <geometry>
-          <mesh filename="package://wamv_description/models/propeller/mesh/propeller.dae"/>
+          <mesh filename="package://wamv_description/models/propeller/mesh/propeller.dae" />
         </geometry>
       </visual>
@@ -39,20 +39,20 @@
       </collision>
       <inertial>
-        <mass value="0.5"/>
-        <inertia ixx="0.008545" ixy="0.0" ixz="0.0" iyy="0.008545" iyz="0.0" izz="0.0144"/>
+        <mass value="0.5" />
+        <inertia ixx="0.008545" ixy="0.0" ixz="0.0" iyy="0.008545" iyz="0.0" izz="0.0144" />
       </inertial>
     </link>
     <joint name="${prefix}_chasis_engine_joint" type="revolute">
-      <axis xyz="0 0 1"/>
-      <limit lower="${-pi}" upper="${pi}" effort="10" velocity="10"/>
-      <origin xyz="${position}" rpy="${orientation}"/>
-      <parent link="base_link"/>
-      <child link="${prefix}_engine_link"/>
+      <axis xyz="0 0 1" />
+      <limit lower="${-pi}" upper="${pi}" effort="10" velocity="10" />
+      <origin xyz="${position}" rpy="${orientation}" />
+      <parent link="base_link" />
+      <child link="${prefix}_engine_link" />
     </joint>
     <joint name="${prefix}_engine_propeller_joint" type="continuous">
-      <axis rpy="0 0 0" xyz="1 0 0"/>
-      <parent link="${prefix}_engine_link"/>
-      <child link="${prefix}_propeller_link"/>
-      <origin rpy="0 0 0" xyz="-0.278156 0 -0.509371"/>
+      <axis rpy="0 0 0" xyz="1 0 0" />
+      <parent link="${prefix}_engine_link" />
+      <child link="${prefix}_propeller_link" />
+      <origin rpy="0 0 0" xyz="-0.278156 0 -0.509371" />
       <limit effort="100" velocity="100" />
       <dynamics friction="0.05" damping="0.05" />

File: vrx_ws/src/vrx/wamv_gazebo/urdf/wamv_gazebo.xacro (robot description, xacro)
@@ -1,6 +1,6 @@
-<?xml version="1.0"?>
+<?xml version="1.0" ?>
 <robot xmlns:xacro="http://ros.org/wiki/xacro">
   <!-- Macro to create a WAM-V with dyanmics plugins and a customizeable thruster layout -->
-  <xacro:macro  name="wamv_gazebo" params="thruster_layout">
+  <xacro:macro name="wamv_gazebo" params="thruster_layout">
     <!-- Include macros for dynamics plugins -->
     <xacro:include filename="$(find wamv_gazebo)/urdf/macros.xacro" />
@@ -8,7 +8,7 @@
     <xacro:include filename="$(find wamv_description)/urdf/wamv_base.urdf.xacro" />
     <!-- Thruster Layout -->
-    <xacro:include filename="${thruster_layout}"/>
+    <xacro:include filename="${thruster_layout}" />
     <!-- Attach hydrodynamics plugin -->
-    <xacro:usv_dynamics_gazebo name="wamv_dynamics_plugin"/>
+    <xacro:usv_dynamics_gazebo name="wamv_dynamics_plugin" />
   </xacro:macro>
 </robot>
