Commit message: update boat

File: catkin_ws/src/duckiepond_vehicle/urdf/duckieboat_new.xacro (robot description, xacro)
@@ -26,6 +26,8 @@
     <!-- Attach thrust plugin -->
     <xacro:include filename="$(find duckiepond_vehicle)/urdf/engine.xacro" />
-    <xacro:engine prefix="left" position="0.5 0.4 0.3" />
-    <xacro:engine prefix="right" position="0.5 -0.4 0.3" />
+    <xacro:engine prefix="left_rear" position="-0.3 0.5 0.25" orientation="0.0 0.0 0.785" />
+    <xacro:engine prefix="right_rear" position="-0.3 -0.5 0.25" orientation="0.0 0.0 -0.785" />
+    <xacro:engine prefix="left_front" position="0.8 0.1  0.25" orientation="0.0 0.0 -0.785" />
+    <xacro:engine prefix="right_front" position="0.8 -0.1 0.25" orientation="0.0 0.0 +0.785" />
     <gazebo>
         <plugin name="gazebo_thrust" filename="libusv_gazebo_thrust_plugin.so">
@@ -33,11 +35,13 @@
             <robotNamespace>${namespace}</robotNamespace>
             <xacro:include filename="$(find duckiepond_vehicle)/urdf/gazebo_thruster_config.xacro" />
-            <xacro:gazebo_thruster_config name="left" />
-            <xacro:gazebo_thruster_config name="right" />
+            <xacro:gazebo_thruster_config name="left_rear" />
+            <xacro:gazebo_thruster_config name="right_rear" />
+            <xacro:gazebo_thruster_config name="left_front" />
+            <xacro:gazebo_thruster_config name="right_front" />
         </plugin>
     </gazebo>
     <!-- Attach LiDAR plugin -->
     <xacro:include filename="$(find duckiepond_vehicle)/urdf/lidar.xacro" />
-    <xacro:lidar name="velodyne" type="16_beam"/>
+    <xacro:lidar name="velodyne" type="16_beam" />
     <!-- Attach camera plugin -->
     <xacro:include filename="$(find duckiepond_vehicle)/urdf/usv_gazebo_camera_plugin.xacro" />

File: catkin_ws/src/duckiepond_vehicle/urdf/engine.xacro (robot description, xacro)
@@ -22,5 +22,5 @@
       </collision>
       <inertial>
-        <mass value="2" />
+        <mass value="0.5" />
         <inertia ixx="0.889245" ixy="0.0" ixz="0.0" iyy="0.911125" iyz="0.0" izz="0.078125" />
       </inertial>

File: catkin_ws/src/duckiepond_vehicle/urdf/gazebo_thruster_config.xacro (robot description, xacro)
@@ -9,5 +9,5 @@
       <cmdTopic>${thruster_namespace}${name}_thrust_cmd</cmdTopic>
       <angleTopic>${thruster_namespace}${name}_thrust_angle</angleTopic>
-      <enableAngle>true</enableAngle>
+      <enableAngle>false</enableAngle>
       <!-- Optional Parameters -->
       <mappingType>1</mappingType>

File: catkin_ws/src/duckiepond_vehicle/urdf/usv_gazebo_dynamics_plugin.xacro (robot description, xacro)
@@ -25,5 +25,5 @@
         <!-- General dimensions -->
         <!--<boatArea>2.2</boatArea>-->
-        <hullRadius>0.213</hullRadius>
+        <hullRadius>0.2</hullRadius>
         <boatWidth>0.75</boatWidth>
         <boatLength>1.5</boatLength>
